File: Button/Button.brd (EAGLE design)
At the start: 160 x 100 mm, 23 parts, among them IC1 4040D, IC2 NE555D

Commit message: routed
Parts:
- moved D13 93.5 mm to (27.1, -14.5), turned to 60 degrees
- moved R2 83.7 mm to (-8.23, -28.4), turned to 300 degrees
- moved D3 80.6 mm to (24.2, 15.7), turned to 320 degrees
- moved D4 79.2 mm to (10.4, 26.7), turned to 40 degrees
- moved D8 78.3 mm to (-20.0, 16.0), turned to 130 degrees
- moved R1 77.8 mm to (-20.2, -23.0), turned to 220 degrees
- moved D6 77.8 mm to (8.35, 12.6), turned to 20 degrees
- moved C1 73.7 mm to (-25.2, -17.7), turned to 120 degrees
- moved R4 71.5 mm to (19.1, 11.2), turned to 140 degrees
- moved C2 71.0 mm to (-18.1, -14.8), turned to 140 degrees
- moved D10 68.9 mm to (-14.3, -10.4), turned to 310 degrees
- moved R7 65.9 mm to (-14.9, -4.58), turned to 40 degrees
- moved IC2 65.6 mm to (-4.65, -16.9), turned to 130 degrees
- moved R6 62.8 mm to (-27.7, 11.0), turned to 150 degrees
- moved D7 62.5 mm to (-4.00, -7.00), turned to 310 degrees
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Routing:
- net GND: track 0.00 -> 237.1 mm, vias 0 -> 4
- net VCC: track 0.00 -> 194.7 mm, vias 0 -> 5
- net N$5: track 0.00 -> 62.2 mm
- net SQ_OUT: track 0.00 -> 48.0 mm
- net N$8: track 0.00 -> 46.5 mm, vias 0 -> 2
- net N$11: track 0.00 -> 41.4 mm
- net N$9: track 0.00 -> 39.2 mm, vias 0 -> 2
- net N$13: track 0.00 -> 37.3 mm
- net N$6: track 0.00 -> 33.5 mm, vias 0 -> 2
- net N$12: track 0.00 -> 26.6 mm
- net N$7: track 0.00 -> 24.7 mm
- net N$3: track 0.00 -> 22.0 mm, vias 0 -> 2
- net N$2: track 0.00 -> 20.8 mm
- net N$1: track 0.00 -> 19.3 mm
- net N$4: track 0.00 -> 9.31 mm
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- added copper zone on layer 1, net GND
- added copper zone on layer 16, net GND
Other:
- board size 160 x 100 mm -> 70 x 70 mm
- board text added: "DAT"
