File: Button/Button.sch (EAGLE design)
At the start: 3 parts, among them IC1 4040D, IC2 NE555D

Commit message: update
Parts:
- added C1: 4.7nf, rcl:C-EUC1206
- added C2: 0.01uf, rcl:C-EUC1206
- added R2: 150k, 1%, rcl:R-EU_R1206
- R1: value (none) -> 4k7, 1%
Connections:
- net N$1 renamed SQ_OUT
- new net N$1: C1.2, IC2.THR
- new net N$2: IC2.DIS, R1.1, R2.1
- new net N$3: IC2.TR, R2.2
- new net N$4: C2.1, IC2.CV
- net GND: now also C1.1, C2.2
- net VCC: now also R1.2
Other:
- moved on the sheet: IC1, R1
Changed lines of the file:
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@@
 <part name="IC1" library="40xx" library_urn="urn:adsk.eagle:library:80" deviceset="4040" device="D" package3d_urn="urn:adsk.eagle:package:821/2"/>
 <part name="IC2" library="linear" library_urn="urn:adsk.eagle:library:262" deviceset="*555" device="D" package3d_urn="urn:adsk.eagle:package:16404/2" technology="NE"/>
-<part name="R1" library="rcl" library_urn="urn:adsk.eagle:library:334" deviceset="R-EU_" device="R1206" package3d_urn="urn:adsk.eagle:package:23540/2"/>
+<part name="R1" library="rcl" library_urn="urn:adsk.eagle:library:334" deviceset="R-EU_" device="R1206" package3d_urn="urn:adsk.eagle:package:23540/2" value="4k7, 1%"/>
+<part name="C1" library="rcl" library_urn="urn:adsk.eagle:library:334" deviceset="C-EU" device="C1206" package3d_urn="urn:adsk.eagle:package:23618/2" value="4.7nf"/>
+<part name="R2" library="rcl" library_urn="urn:adsk.eagle:library:334" deviceset="R-EU_" device="R1206" package3d_urn="urn:adsk.eagle:package:23540/2" value="150k, 1%"/>
+<part name="C2" library="rcl" library_urn="urn:adsk.eagle:library:334" deviceset="C-EU" device="C1206" package3d_urn="urn:adsk.eagle:package:23618/2" value="0.01uf"/>
 </parts>
 <sheets>
@@
 </plain>
 <instances>
-<instance part="IC1" gate="A" x="43.18" y="33.02" smashed="yes">
-<attribute name="NAME" x="35.56" y="48.895" size="1.778" layer="95"/>
-<attribute name="VALUE" x="35.56" y="12.7" size="1.778" layer="96"/>
+<instance part="IC1" gate="A" x="68.58" y="43.18" smashed="yes">
+<attribute name="NAME" x="60.96" y="59.055" size="1.778" layer="95"/>
+<attribute name="VALUE" x="60.96" y="22.86" size="1.778" layer="96"/>
 </instance>
 <instance part="IC2" gate="A" x="0" y="38.1" smashed="yes">
@@
 <attribute name="VALUE" x="-7.62" y="25.273" size="1.778" layer="96"/>
 </instance>
-<instance part="R1" gate="G$1" x="-12.7" y="17.78" smashed="yes">
-<attribute name="NAME" x="-16.51" y="19.2786" size="1.778" layer="95"/>
-<attribute name="VALUE" x="-16.51" y="14.478" size="1.778" layer="96"/>
+<instance part="R1" gate="G$1" x="25.4" y="40.64" smashed="yes">
+<attribute name="NAME" x="21.59" y="42.1386" size="1.778" layer="95"/>
+<attribute name="VALUE" x="21.59" y="37.338" size="1.778" layer="96"/>
+</instance>
+<instance part="C1" gate="G$1" x="27.94" y="35.56" smashed="yes" rot="R270">
+<attribute name="NAME" x="28.321" y="34.036" size="1.778" layer="95" rot="R270"/>
+<attribute name="VALUE" x="23.241" y="34.036" size="1.778" layer="96" rot="R270"/>
+</instance>
+<instance part="R2" gate="G$1" x="25.4" y="48.26" smashed="yes">
+<attribute name="NAME" x="21.59" y="49.7586" size="1.778" layer="95"/>
+<attribute name="VALUE" x="21.59" y="44.958" size="1.778" layer="96"/>
+</instance>
+<instance part="C2" gate="G$1" x="-15.24" y="35.56" smashed="yes" rot="R270">
+<attribute name="NAME" x="-14.859" y="34.036" size="1.778" layer="95" rot="R270"/>
+<attribute name="VALUE" x="-19.939" y="34.036" size="1.778" layer="96" rot="R270"/>
 </instance>
 </instances>
@@
 </busses>
 <nets>
-<net name="N$1" class="0">
-<segment>
-<pinref part="IC2" gate="A" pin="Q"/>
-<pinref part="IC1" gate="A" pin="P1"/>
-<wire x1="10.16" y1="45.72" x2="30.48" y2="45.72" width="0.1524" layer="91"/>
-</segment>
-</net>
 <net name="VCC" class="0">
 <segment>
@@
 <segment>
 <pinref part="IC2" gate="A" pin="V+"/>
-<wire x1="10.16" y1="30.48" x2="17.78" y2="30.48" width="0.1524" layer="91"/>
-<label x="17.78" y="30.48" size="1.27" layer="95" xref="yes"/>
+<wire x1="10.16" y1="30.48" x2="12.7" y2="30.48" width="0.1524" layer="91"/>
+<label x="12.7" y="30.48" size="1.27" layer="95" xref="yes"/>
+</segment>
+<segment>
+<pinref part="R1" gate="G$1" pin="2"/>
+<wire x1="30.48" y1="40.64" x2="33.02" y2="40.64" width="0.1524" layer="91"/>
+<label x="33.02" y="40.64" size="1.27" layer="95" xref="yes"/>
 </segment>
 </net>
@@
 <label x="-17.78" y="30.48" size="1.27" layer="95" rot="R180" xref="yes"/>
 </segment>
+<segment>
+<pinref part="C1" gate="G$1" pin="1"/>
+<wire x1="30.48" y1="35.56" x2="33.02" y2="35.56" width="0.1524" layer="91"/>
+<label x="33.02" y="35.56" size="1.27" layer="95" xref="yes"/>
+</segment>
+<segment>
+<pinref part="C2" gate="G$1" pin="2"/>
+<wire x1="-20.32" y1="35.56" x2="-22.86" y2="35.56" width="0.1524" layer="91"/>
+<label x="-22.86" y="35.56" size="1.27" layer="95" rot="R180" xref="yes"/>
+</segment>
 </net>
+<net name="N$2" class="0">
+<segment>
+<pinref part="IC2" gate="A" pin="DIS"/>
+<pinref part="R1" gate="G$1" pin="1"/>
+<wire x1="20.32" y1="40.64" x2="17.78" y2="40.64" width="0.1524" layer="91"/>
+<pinref part="R2" gate="G$1" pin="1"/>
+<wire x1="17.78" y1="40.64" x2="10.16" y2="40.64" width="0.1524" layer="91"/>
+<wire x1="17.78" y1="40.64" x2="17.78" y2="48.26" width="0.1524" layer="91"/>
+<wire x1="17.78" y1="48.26" x2="20.32" y2="48.26" width="0.1524" layer="91"/>
+<junction x="17.78" y="40.64"/>
+</segment>
+</net>
+<net name="SQ_OUT" class="0">
+<segment>
+<pinref part="IC2" gate="A" pin="Q"/>
+<wire x1="12.7" y1="45.72" x2="10.16" y2="45.72" width="0.1524" layer="91"/>
+<label x="12.7" y="45.72" size="1.27" layer="95" rot="R90" xref="yes"/>
+</segment>
+<segment>
+<pinref part="IC1" gate="A" pin="P1"/>
+<wire x1="55.88" y1="55.88" x2="53.34" y2="55.88" width="0.1524" layer="91"/>
+<label x="53.34" y="55.88" size="1.27" layer="95" rot="R90" xref="yes"/>
+</segment>
+</net>
+<net name="N$1" class="0">
+<segment>
+<pinref part="IC2" gate="A" pin="THR"/>
+<pinref part="C1" gate="G$1" pin="2"/>
+<wire x1="10.16" y1="35.56" x2="22.86" y2="35.56" width="0.1524" layer="91"/>
+</segment>
+</net>
+<net name="N$3" class="0">
+<segment>
+<pinref part="R2" gate="G$1" pin="2"/>
+<wire x1="30.48" y1="48.26" x2="33.02" y2="48.26" width="0.1524" layer="91"/>
+<wire x1="33.02" y1="48.26" x2="33.02" y2="60.96" width="0.1524" layer="91"/>
+<wire x1="33.02" y1="60.96" x2="-10.16" y2="60.96" width="0.1524" layer="91"/>
+<pinref part="IC2" gate="A" pin="TR"/>
+<wire x1="-10.16" y1="60.96" x2="-10.16" y2="45.72" width="0.1524" layer="91"/>
+</segment>
+</net>
+<net name="N$4" class="0">
+<segment>
+<pinref part="C2" gate="G$1" pin="1"/>
+<pinref part="IC2" gate="A" pin="CV"/>
+<wire x1="-12.7" y1="35.56" x2="-10.16" y2="35.56" width="0.1524" layer="91"/>
+</segment>
+</net>

Commit message: 0
Parts:
- added U$1: BATTHLDR1025-7, BATT_HLDR_COIN:BATTHLDR1025-7
Connections:
- new net +VBAT: U$1.+
- net GND: now also U$1.-
Changed lines of the file:
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@@
 <part name="R2" library="rcl" library_urn="urn:adsk.eagle:library:334" deviceset="R-EU_" device="R1206" package3d_urn="urn:adsk.eagle:package:23540/2" value="150k, 1%"/>
 <part name="C2" library="rcl" library_urn="urn:adsk.eagle:library:334" deviceset="C-EU" device="C1206" package3d_urn="urn:adsk.eagle:package:23618/2" value="0.01uf"/>
+<part name="U$1" library="BATT_HLDR_COIN" deviceset="BATTHLDR1025-7" device=""/>
 </parts>
 <sheets>
@@
 <attribute name="NAME" x="-14.859" y="34.036" size="1.778" layer="95" rot="R270"/>
 <attribute name="VALUE" x="-19.939" y="34.036" size="1.778" layer="96" rot="R270"/>
+</instance>
+<instance part="U$1" gate="G$1" x="55.88" y="5.08" smashed="yes">
+<attribute name="NAME" x="52.07" y="10.16" size="1.778" layer="95"/>
+<attribute name="VALUE" x="52.07" y="-1.27" size="1.778" layer="96"/>
 </instance>
 </instances>
@@
 <wire x1="-20.32" y1="35.56" x2="-22.86" y2="35.56" width="0.1524" layer="91"/>
 <label x="-22.86" y="35.56" size="1.27" layer="95" rot="R180" xref="yes"/>
+</segment>
+<segment>
+<pinref part="U$1" gate="G$1" pin="-"/>
+<wire x1="58.42" y1="5.08" x2="60.96" y2="5.08" width="0.1524" layer="91"/>
+<label x="60.96" y="5.08" size="1.27" layer="95" xref="yes"/>
 </segment>
 </net>
@@
 </segment>
 </net>
+<net name="+VBAT" class="0">
+<segment>
+<pinref part="U$1" gate="G$1" pin="+"/>
+<wire x1="50.8" y1="5.08" x2="48.26" y2="5.08" width="0.1524" layer="91"/>
+<label x="48.26" y="5.08" size="1.27" layer="95" rot="R180" xref="yes"/>
+</segment>
+</net>

Commit message: workshop part 2
Parts:
- added D1, D10, D2, D3, D4, D5, D6, D7, D8, D9: (no value), SparkFun-LED:LED1206
- added D13: (no value), adafruit:DIODESMA
- added R3, R4, R5, R6, R7: 680, 1%, rcl:R-EU_R1206
Connections:
- new net N$10: IC1A.Q6, R5.1
- new net N$11: D7.C, D8.A, R6.2
- new net N$12: IC1A.Q10, R6.1
- new net N$13: D10.A, D9.C, R7.2
- new net N$14: IC1A.Q12, R7.1
- new net N$5: D1.C, D2.A, R3.2
- new net N$6: IC1A.Q2, R3.1
- new net N$7: D3.C, D4.A, R4.2
- new net N$8: IC1A.Q4, R4.1
- new net N$9: D5.C, D6.A, R5.2
- net +VBAT: now also D13.A
- net GND: now also D10.C, D2.C, D4.C, D6.C, D8.C, IC1A.RES, IC1P.VSS
- net VCC: now also D1.A, D13.C, D3.A, D5.A, D7.A, D9.A, IC1P.VDD
Other:
- moved on the sheet: IC1, U$1

Commit message: routed
Other:
- moved on the sheet: IC1P
Changed lines of the file:
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@@
 <?xml version="1.0" encoding="utf-8"?>
 <!DOCTYPE eagle SYSTEM "eagle.dtd">
-<eagle version="9.3.2">
+<eagle version="9.6.2">
 <drawing>
 <settings>
@@
 </variantdefs>
 <classes>
-<class number="0" name="default" width="0" drill="0">
+<class number="0" name="default" width="0.3048" drill="0.3048">
+<clearance class="0" value="0.3048"/>
 </class>
 </classes>
@@
 <attribute name="VALUE" x="-74.93" y="39.37" size="1.778" layer="96" rot="R180"/>
 </instance>
-<instance part="IC1" gate="P" x="68.58" y="78.74" smashed="yes" rot="R270">
-<attribute name="NAME" x="67.945" y="77.47" size="1.778" layer="95" rot="R270"/>
+<instance part="IC1" gate="P" x="76.2" y="78.74" smashed="yes" rot="R270">
+<attribute name="NAME" x="75.565" y="77.47" size="1.778" layer="95" rot="R270"/>
 </instance>
 <instance part="D1" gate="G$1" x="121.92" y="60.96" smashed="yes" rot="R270">
@@
 <segment>
 <pinref part="IC1" gate="P" pin="VDD"/>
-<wire x1="76.2" y1="78.74" x2="78.74" y2="78.74" width="0.1524" layer="91"/>
-<label x="78.74" y="78.74" size="1.27" layer="95" xref="yes"/>
+<wire x1="83.82" y1="78.74" x2="86.36" y2="78.74" width="0.1524" layer="91"/>
+<label x="86.36" y="78.74" size="1.27" layer="95" xref="yes"/>
 </segment>
 <segment>
@@
 <segment>
 <pinref part="IC1" gate="P" pin="VSS"/>
-<wire x1="60.96" y1="78.74" x2="58.42" y2="78.74" width="0.1524" layer="91"/>
-<label x="58.42" y="78.74" size="1.27" layer="95" rot="R180" xref="yes"/>
+<wire x1="68.58" y1="78.74" x2="66.04" y2="78.74" width="0.1524" layer="91"/>
+<label x="66.04" y="78.74" size="1.27" layer="95" rot="R180" xref="yes"/>
 </segment>
 <segment>
@@
 </sheet>
 </sheets>
+<errors>
+</errors>
 </schematic>
 </drawing>
